Commit message: Get a working roslaunch sim.

File: src/gudrun_sim/urdf/gudrun.urdf.xacro (robot description, xacro)
@@ -7,4 +7,6 @@
 	<xacro:property name="length" value="0.5"/>
 	<xacro:property name="height" value="0.125"/>
+	<xacro:property name="wheel_width" value="0.0625" />
+	<xacro:property name="wheel_radius" value="0.0625" />
 	<link name="base_link">
 		<visual>
@@ -23,6 +25,4 @@
 		</inertial>
 	</link>
-	<xacro:property name="wheel_width" value="0.0625" />
-	<xacro:property name="wheel_radius" value="0.0625" />
 	<xacro:macro name="wheel" params="suffix *origin">
 		<link name="wheel_${suffix}">
@@ -56,7 +56,14 @@
 			</actuator>
 			<joint name="base_link_to_wheel_${suffix}">
-				<hardwareInterface>PositionJointInterface</hardwareInterface>
+				<hardwareInterface>hardware_interface/VelocityJointInterface</hardwareInterface>
 			</joint>
 		</transmission>
+		<gazebo reference="${suffix}_wheel">
+			<mu1 value="200.0"/>
+			<mu2 value="100.0"/>
+			<kp value="10000000.0" />
+			<kd value="1.0" />
+			<material>Gazebo/Grey</material>
+		</gazebo>
 	</xacro:macro>
 	<xacro:wheel suffix="left_front">
